Commit message: SO-101: hardware arming gate, consistent camera model, policy episodes
- The hardware stack routes policy commands through so101_hil_guard,
  disarmed by default and gated on fresh joint feedback.
- One camera model: the scenario camera drives Isaac, CameraInfo (69 deg
  HFOV, fx 465.6), the URDF and TF, and the validator checks against it.
  Isaac now publishes its real render (it published a synthetic
  placeholder) with a usable near clip and a pose that sees the task.
- Reset the policy server at start, after feedback gaps and on task
  change; command rate configurable to the dataset fps.
- Send native-resolution or letterboxed images instead of squashing 4:3
  frames into a square.
- Reject non-finite commands in every simulator, the Gazebo relay and the
  CBF controller; the HIL guard survives a short JointState.
- Metrics: latency, observation age, saturation, joint-limit violations and
  ground-truth use are measured; unmeasured collisions fail acceptance.
- LeRobot units: reject normalised [-100, 100] data; per-joint sign/offset
  mapping (placeholder values until calibrated on the arm).
- Genesis copies CUDA tensors to the host and keeps system site-packages.
- Pin Isaac-GR00T (d2b7e75) and lerobot (0.6.0), pass the policy port
  through, drop the gym service that could not run.

Co-Authored-By: Claude Opus 5.5 <noreply@anthropic.com>

File: systems/so101/urdf/so101.urdf (robot description, URDF)
Before this commit: robot so101, 12 links, 11 joints
Joints:
- joint base_to_groot_camera: origin xyz=0.24 -0.28 0.34 rpy=0.0 0.72 2.36 -> xyz=0.17 -0.52 0.4665 rpy=0.0 0.785 1.449

File: systems/so101/urdf/so101.urdf.xacro (robot description, xacro)
@@ -85,11 +85,15 @@
     <parent link="gripper_base_link"/><child link="fixed_jaw_link"/>
   </joint>
+  <!-- The camera body sits behind the lens so the simulator camera, rendered
+       at this link's origin, does not look out from inside it. -->
   <link name="groot_camera_link">
-    <visual><geometry><box size="0.035 0.025 0.025"/></geometry><material name="so101_black"/></visual>
-    <collision><geometry><box size="0.035 0.025 0.025"/></geometry></collision>
+    <visual><origin xyz="-0.02 0 0"/><geometry><box size="0.035 0.025 0.025"/></geometry><material name="so101_black"/></visual>
+    <collision><origin xyz="-0.02 0 0"/><geometry><box size="0.035 0.025 0.025"/></geometry></collision>
   </link>
+  <!-- Must equal the scenario camera pose (systems/so101/scenarios/picking_table.json
+       "camera") relative to base_link; checked by validate_calibration_and_dataset.py. -->
   <joint name="base_to_groot_camera" type="fixed">
     <parent link="base_link"/><child link="groot_camera_link"/>
-    <origin xyz="0.24 -0.28 0.34" rpy="0.0 0.72 2.36"/>
+    <origin xyz="0.17 -0.52 0.4665" rpy="0.0 0.785 1.449"/>
   </joint>
   <link name="groot_camera_rgb_optical_frame"/>

Commit message: SO-101: one joint-limit table matching the arm's real range
systems/so101/config/joint_limits.json is now the single source of truth
for joint position limits. The xacro loads it, and so101_common, the
GR00T scripts and the SmolVLA server read it from the /workspace/systems
mount. The values are TheRobotStudio's so101_new_calib.urdf limits mapped
into this URDF's straight-up zero with lerobot_joint_mapping.json, so a
LeRobot-calibrated arm's full travel fits (the elbow is -22.9..170.7 deg,
not +/-100 deg).

The SmolVLA server and the GR00T dataset normaliser warn about, or reject,
checkpoint and dataset ranges that fall outside these limits once mapped.
The six controller and HIL-guard services that load the limits now mount
systems/.

Co-Authored-By: Claude Opus 5.5 <noreply@anthropic.com>

File: systems/so101/urdf/so101.urdf (robot description, URDF)
Before this commit: robot so101, 12 links, 11 joints
Joints:
- joint elbow_flex: limit lower=-1.7453 upper=1.7453 effort=6.0 velocity=3.0 -> lower=-0.40021 upper=2.9798 effort=6.0 velocity=3.0
- joint shoulder_lift: limit lower=-1.7453 upper=1.7453 effort=6.0 velocity=3.0 -> lower=-1.50099 upper=1.98968 effort=6.0 velocity=3.0
- joint shoulder_pan: limit lower=-1.9199 upper=1.9199 effort=6.0 velocity=3.0 -> lower=-1.91986 upper=1.91986 effort=6.0 velocity=3.0
- joint wrist_flex: limit lower=-1.6581 upper=1.6581 effort=3.0 velocity=4.0 -> lower=-1.62141 upper=1.69472 effort=3.0 velocity=4.0
- joint wrist_roll: limit lower=-2.7439 upper=2.7439 effort=3.0 velocity=4.0 -> lower=-2.84121 upper=2.74385 effort=3.0 velocity=4.0

File: systems/so101/urdf/so101.urdf.xacro (robot description, xacro)
@@ -19,4 +19,12 @@
     </link>
   </xacro:macro>
+  <!-- Joint position limits come from their single source of truth,
+       systems/so101/config/joint_limits.json (see the derivation there).
+       A relative load_yaml path resolves against this file's directory. -->
+  <xacro:property name="joint_limits" value="${xacro.load_yaml('../config/joint_limits.json')['joints']}"/>
+  <xacro:macro name="joint_limit" params="name effort velocity">
+    <limit lower="${joint_limits[name]['lower']}" upper="${joint_limits[name]['upper']}"
+           effort="${effort}" velocity="${velocity}"/>
+  </xacro:macro>
   <link name="world"/>
   <xacro:box_link name="base_link" sx="0.12" sy="0.12" sz="0.045" mass="0.42" color="so101_black"/>
@@ -28,5 +36,5 @@
     <parent link="base_link"/><child link="shoulder_link"/>
     <origin xyz="0 0 0.065"/><axis xyz="0 0 1"/>
-    <limit lower="-1.9199" upper="1.9199" effort="6.0" velocity="3.0"/>
+    <xacro:joint_limit name="shoulder_pan" effort="6.0" velocity="3.0"/>
     <dynamics damping="0.08" friction="0.02"/>
   </joint>
@@ -39,5 +47,5 @@
     <parent link="shoulder_link"/><child link="upper_arm_link"/>
     <origin xyz="0 0 0.045"/><axis xyz="0 1 0"/>
-    <limit lower="-1.7453" upper="1.7453" effort="6.0" velocity="3.0"/>
+    <xacro:joint_limit name="shoulder_lift" effort="6.0" velocity="3.0"/>
     <dynamics damping="0.08" friction="0.02"/>
   </joint>
@@ -50,5 +58,5 @@
     <parent link="upper_arm_link"/><child link="forearm_link"/>
     <origin xyz="0 0 0.14"/><axis xyz="0 1 0"/>
-    <limit lower="-1.7453" upper="1.7453" effort="6.0" velocity="3.0"/>
+    <xacro:joint_limit name="elbow_flex" effort="6.0" velocity="3.0"/>
     <dynamics damping="0.07" friction="0.02"/>
   </joint>
@@ -57,5 +65,5 @@
     <parent link="forearm_link"/><child link="wrist_pitch_link"/>
     <origin xyz="0 0 0.13"/><axis xyz="0 1 0"/>
-    <limit lower="-1.6581" upper="1.6581" effort="3.0" velocity="4.0"/>
+    <xacro:joint_limit name="wrist_flex" effort="3.0" velocity="4.0"/>
     <dynamics damping="0.05" friction="0.01"/>
   </joint>
@@ -64,5 +72,5 @@
     <parent link="wrist_pitch_link"/><child link="wrist_roll_link"/>
     <origin xyz="0 0 0.055"/><axis xyz="0 0 1"/>
-    <limit lower="-2.7439" upper="2.7439" effort="3.0" velocity="4.0"/>
+    <xacro:joint_limit name="wrist_roll" effort="3.0" velocity="4.0"/>
     <dynamics damping="0.04" friction="0.01"/>
   </joint>
@@ -75,5 +83,5 @@
     <parent link="gripper_base_link"/><child link="gripper_jaw_link"/>
     <origin xyz="0.025 0 0.035"/><axis xyz="1 0 0"/>
-    <limit lower="0.0" upper="0.04" effort="2.0" velocity="0.15"/>
+    <xacro:joint_limit name="gripper" effort="2.0" velocity="0.15"/>
     <dynamics damping="0.05" friction="0.01"/>
   </joint>

Commit message: SO-101 scene: one source of truth for heights, the D435i's real camera
The pick-and-place scene was inconsistent across simulators and with the
printed station:
- the arm spawned 31 mm above the table and its mount box overlapped its
  base by 29 mm;
- objects floated at 0.46 m and bins at 0.4325 m (Isaac kept them there,
  Gazebo dropped them);
- the calibration board floated;
- Gazebo had a hard-coded spawn height and a rear panel no other simulator
  had;
- Genesis did not load the scene at all.

systems/so101/scenarios/picking_table.json is now the only place heights
are written:
- The arm sits on a 31 mm riser (spawn 0.431 m); bins, objects, the
  occluder and the calibration board (in its printed feet) rest on the
  table.
- Every entry names what it rests on, and so101_common.scene_support_errors
  flags anything floating, sunk or overlapping. Tests, the dataset
  validator and Isaac and Genesis at start-up run it.
- The Gazebo world is generated from the scenario (scenario_world.py; a test
  fails if it is stale), gazebo.launch.py spawns at its robot_spawn, and
  the camera constants, table frame (0.400 m) and the scorer's minimum
  height read from it.
- A test fails if a script or composition hard-codes a scene height.

The simulated camera is now the RealSense D435i colour stream:
- 640x360, 69.4 x 42.5 deg, at the printed head's recommended 48.5 deg
  pitch; every bin and object is within 88 % of the half-image.
- The pose rotates about the head's existing pivot, so the printed parts
  are unchanged.
- The hardware compositions request the same 640x360 profile.
- Policies trained on the old 4:3 view need retraining or a warp; the
  READMEs say how.

The scripted demo grasps with the jaws turned sideways, 5 mm above the
table: the old pose only cleared because the objects floated 60 mm up.
Isaac solves it (2.4 mm place error); Gazebo's simplified gripper misses the
grasp (it never grasped before either), and Genesis's grasp is not
physical. Genesis also ran at 0.1x real time until its frames went out as
byte arrays (Humble's rclpy spent 90 ms checking each).

Co-Authored-By: Claude Opus 5.5 <noreply@anthropic.com>

File: systems/so101/urdf/so101.urdf (robot description, URDF)
Before this commit: robot so101, 12 links, 11 joints
Joints:
- joint base_to_groot_camera: origin xyz=0.17 -0.52 0.4665 rpy=0.0 0.785 1.449 -> xyz=0.1697563 -0.5219908 0.4646126 rpy=0.0 0.8464847 1.449

File: systems/so101/urdf/so101.urdf.xacro (robot description, xacro)
@@ -103,5 +103,5 @@
   <joint name="base_to_groot_camera" type="fixed">
     <parent link="base_link"/><child link="groot_camera_link"/>
-    <origin xyz="0.17 -0.52 0.4665" rpy="0.0 0.785 1.449"/>
+    <origin xyz="0.1697563 -0.5219908 0.4646126" rpy="0.0 0.8464847 1.449"/>
   </joint>
   <link name="groot_camera_rgb_optical_frame"/>
