Commit message: RACECAR Neo: SI Ackermann commands, URDF frames, simulator vehicle model
- /ackermann_cmd is SI (m/s, rad); steering comes from the requested
  twist's curvature, and NaN twists are dropped.
- Bridge: create the racecar on the main thread (the library's signal()
  call failed in a thread, so it never connected); odometry counts encoder
  ticks instead of rounding the integrated pose; IMU converted from Unity
  axes; camera intrinsics from the simulator's 42.5 deg vertical FOV.
- Simulator vehicle model: the RacecarSim car's wheelbase is 0.225 m (wheel
  colliders at +-1.125 Unity units, 1 unit = 0.1 m), not the hardware
  0.33 m. The bridge, the simulator's converter and URDF sim_geometry use
  it, so Nav2's curvature reaches the simulator unchanged (it was ~47%
  tighter). Nav2's 0.75 m turning radius is unchanged; the simulated car
  can turn at 0.62 m.
- The URDF is the single source of sensor frames (racecarneo/ prefix),
  published by robot_state_publisher in both stacks.
- Hardware wiring: nvblox topics are launch arguments, RealSense topics
  match /camera/color/*.
- NiceGUI shows the map-frame pose and no longer crashes on load.
- Pin the simulator (v2.8.3), racecar library, Depth-Anything-V2 and its
  weights (sha256), torch, nicegui and nvblox assets.
- Foxglove services run foxglove_bridge.

Co-Authored-By: Claude Opus 5.5 <noreply@anthropic.com>

File: systems/racecarneo/urdf/racecarneo.urdf.xacro (robot description, xacro)
@@ -1,4 +1,25 @@
 <?xml version="1.0"?>
+<!--
+  RACECAR Neo frame model and the single source of sensor extrinsics for
+  both the simulator and the hardware stack: robot_state_publisher publishes
+  it in compositions/racecarneo.yaml and racecarneo_hardware.yaml. Frame
+  names match systems/racecarneo/config/topics.yaml.
+  The hardware offsets are the simulator bridge's long-standing values, not
+  measurements of a physical car; measure and update them for hardware.
+  sim_geometry:=true selects the mounts of the RacecarSim v2.8.3 car, which
+  is smaller (0.225 m wheelbase): read from its Racecar prefab
+  (sharedassets2.assets), Lidar at (0, 1.25, 0) and ColorCamera/DepthCamera at
+  (0, 1.45, 1.0) Unity units, where 1 unit = 0.1 m (the simulator scales
+  lidar and depth distances by 10 to report centimetres).
+-->
 <robot xmlns:xacro="http://www.ros.org/wiki/xacro" name="racecarneo">
+  <!--
+    The simulator has no camera driver, so the URDF publishes the optical
+    frames too. On hardware the RealSense driver (tf_prefix racecarneo/)
+    publishes racecarneo/camera_link -> optical frames from its factory
+    calibration, so run xacro with camera_optical_frames:=false there.
+  -->
+  <xacro:arg name="camera_optical_frames" default="true"/>
+  <xacro:arg name="sim_geometry" default="false"/>
   <link name="base_link">
     <visual>
@@ -17,26 +38,50 @@
     </inertial>
   </link>
-  <link name="lidar_link"/>
-  <joint name="lidar_joint" type="fixed">
-    <parent link="base_link"/>
-    <child link="lidar_link"/>
-    <origin xyz="0.02 0 0.16" rpy="0 0 0"/>
-  </joint>
-  <link name="camera_color_optical_frame"/>
-  <joint name="camera_color_joint" type="fixed">
-    <parent link="base_link"/>
-    <child link="camera_color_optical_frame"/>
-    <origin xyz="0.16 0 0.13" rpy="-1.57079632679 0 -1.57079632679"/>
-  </joint>
-  <link name="camera_depth_optical_frame"/>
-  <joint name="camera_depth_joint" type="fixed">
-    <parent link="camera_color_optical_frame"/>
-    <child link="camera_depth_optical_frame"/>
-    <origin xyz="0 0 0" rpy="0 0 0"/>
-  </joint>
-  <link name="imu_link"/>
+  <link name="racecarneo/lidar_link"/>
+  <!-- Camera body, x forward / y left / z up (RealSense camera_link). -->
+  <link name="racecarneo/camera_link"/>
+  <xacro:unless value="$(arg sim_geometry)">
+    <joint name="lidar_joint" type="fixed">
+      <parent link="base_link"/>
+      <child link="racecarneo/lidar_link"/>
+      <origin xyz="0.08 0 0.18" rpy="0 0 0"/>
+    </joint>
+    <joint name="camera_joint" type="fixed">
+      <parent link="base_link"/>
+      <child link="racecarneo/camera_link"/>
+      <origin xyz="0.18 0 0.22" rpy="0 0 0"/>
+    </joint>
+  </xacro:unless>
+  <xacro:if value="$(arg sim_geometry)">
+    <joint name="lidar_joint" type="fixed">
+      <parent link="base_link"/>
+      <child link="racecarneo/lidar_link"/>
+      <origin xyz="0 0 0.125" rpy="0 0 0"/>
+    </joint>
+    <joint name="camera_joint" type="fixed">
+      <parent link="base_link"/>
+      <child link="racecarneo/camera_link"/>
+      <origin xyz="0.10 0 0.145" rpy="0 0 0"/>
+    </joint>
+  </xacro:if>
+  <!-- Optical frames: z forward, x right, y down (REP-103). -->
+  <xacro:if value="$(arg camera_optical_frames)">
+    <link name="racecarneo/camera_color_optical_frame"/>
+    <joint name="camera_color_optical_joint" type="fixed">
+      <parent link="racecarneo/camera_link"/>
+      <child link="racecarneo/camera_color_optical_frame"/>
+      <origin xyz="0 0 0" rpy="-1.57079632679 0 -1.57079632679"/>
+    </joint>
+    <link name="racecarneo/camera_depth_optical_frame"/>
+    <joint name="camera_depth_optical_joint" type="fixed">
+      <parent link="racecarneo/camera_link"/>
+      <child link="racecarneo/camera_depth_optical_frame"/>
+      <origin xyz="0 0 0" rpy="-1.57079632679 0 -1.57079632679"/>
+    </joint>
+  </xacro:if>
+  <link name="racecarneo/imu_link"/>
   <joint name="imu_joint" type="fixed">
     <parent link="base_link"/>
-    <child link="imu_link"/>
+    <child link="racecarneo/imu_link"/>
     <origin xyz="0 0 0.08" rpy="0 0 0"/>
   </joint>

Commit message: Work in progress: RACECAR Turret Isaac evaluation, depth, tracking and BlueOS fixes
A snapshot, at the user's request, of work whose agents are still running.
Every check passes on this tree: pytest, ruff, docker compose config for
every composition, the env-default check and CI's shellcheck. Each area's
final results follow in its own commit.

RACECAR Turret Isaac evaluation (complete):
- applications/isaac/scripts/racecar_turret_*.py: an Ackermann car with
  lidar, RGB-D, IMU, wheel odometry and the turret in a 20 x 15 m arena
  with walking people;
- compositions/racecar_turret_isaac.yaml: SLAM Toolbox, Nav2, nvblox and
  the turret tracker on simulation time;
- tools/racecar_turret_{evaluator,scorer}.py and
  tools/racecar_turret_isaac_test.sh.
Measured: the course completed in every run with no collisions; while
following the target, compensation and lead cut the aim error's p95 from
3.5-3.8 deg to 1.4-1.5 deg. The assets pass launcher:=false to the turret
macro.

RACECAR depth (in progress): Depth Anything's vkitti metric model read the
RACECAR's depth about 8.6x too far from its 0.22 m camera. This adds metric
depth variants and per-frame scale alignment in depthanything_pkg, an
accuracy tool, nvblox settings for Isaac, the RacecarSim camera's measured
height and pitch in the URDF, and a costmap coverage check. The evaluation
re-run and the hardware recommendation are still to come.

Aerial tracking (in progress):
- the tracker's lost and handover timeouts on the node clock (simulation
  time in the simulators);
- the Genesis references removed from the tracking files;
- the UI fixes.
The Gazebo and Isaac re-runs against the scorer are still to come.

BlueOS on the Raspberry Pi 5 (in progress), from testing on the real Pi:
- rosbridge moves to port 9092, because BlueOS's Cable Guy holds 9090,
  with host IPC and /dev/shm so Fast DDS delivers messages to it;
- the rangefinder is reached through device cgroup rules instead of a
  devices: entry, so the aerodrone stack starts without the adapter
  plugged in and picks it up when it appears;
- docs and a test.
The MAVROS link over BlueOS's internal TCP port, the cache seeds and the
OAK-1 retry are still to come.

Not included: the aerodrone's downward launcher parts, whose build is not
finished.

Co-Authored-By: Claude Opus 5.5 <noreply@anthropic.com>

File: systems/racecarneo/urdf/racecarneo.urdf.xacro (robot description, xacro)
@@ -14,5 +14,6 @@
   (sharedassets2.assets), Lidar at (0, 1.25, 0) and ColorCamera/DepthCamera at
   (0, 1.45, 1.0) Unity units, where 1 unit = 0.1 m (the simulator scales
-  lidar and depth distances by 10 to report centimetres).
+  lidar and depth distances by 10 to report centimetres); the camera's
+  height and pitch are measured from its depth instead (below).
 -->
 <robot xmlns:xacro="http://www.ros.org/wiki/xacro" name="racecarneo">
@@ -62,8 +63,14 @@
       <origin xyz="0 0 0.125" rpy="0 0 0"/>
     </joint>
+    <!-- The camera as the simulator renders it: its depth puts the floor
+         0.120 m below the camera, pitched 0.81 deg up (Demo World, 195
+         frames; the floor then within 2.4 mm of z = 0 from 0.3 to 4 m;
+         applications/racecarneo/README.md, "Depth for nvblox"), not at the
+         prefab's level 0.145 m, which lifted the near floor into nvblox's
+         0.02 m obstacle band. -->
     <joint name="camera_joint" type="fixed">
       <parent link="base_link"/>
       <child link="racecarneo/camera_link"/>
-      <origin xyz="0.10 0 0.145" rpy="0 0 0"/>
+      <origin xyz="0.10 0 0.120" rpy="0 -0.0141 0"/>
     </joint>
   </xacro:if>
